File: doc/circuit/circuit.brd (EAGLE design)
At the start: 63.2 x 45.7 mm, 23 parts, among them U1 LPC1114FN28/102

Commit message: Added docs.
Parts:
- CDS+, CDS-, CLKOUT, GND, IR+, IR-, RESET, RXD, TXD, VCC: value WIREPAD2,54/1,0 -> WIREPAD2,15/1,0; device wirepad:2,54/1,0 -> wirepad:2,15/1,0
- R2: value 100 -> 1k
- moved S2 38.3 mm to (7.62, 43.2), turned to 180 degrees
- moved TXD 7.18 mm to (55.9, 30.5)
- moved RXD 3.59 mm to (58.4, 30.5)
- moved CLKOUT 2.54 mm to (35.6, 30.5)
- moved RESET 2.54 mm to (38.1, 30.5)
- moved CDS+ 2.54 mm to (55.9, 5.08)
- moved CDS- 2.54 mm to (55.9, 7.62)
- moved IR+ 2.54 mm to (58.4, 7.62)
- moved IR- 2.54 mm to (58.4, 5.08)
- moved LED1 1.80 mm to (49.5, 40.6), turned to 180 degrees
- moved S1 1.14 mm to (59.1, 41.0)
- moved G1 0.64 mm to (12.7, 19.7), turned to 0 degrees
Routing:
- net VCC: track 135.0 -> 180.9 mm
- net GND: track 149.3 -> 176.6 mm
- net GND2: track 12.7 -> 2.54 mm
- net N$5: track 24.1 -> 33.0 mm
- net VCC3: track 7.62 -> 2.54 mm
- net N$4: track 5.08 -> 2.54 mm
- net N$3: track 5.08 -> 2.54 mm
- net VCC1: track 17.8 -> 15.2 mm
- net N$9: track 16.3 -> 13.8 mm, vias 0 -> 2
- net N$2: track 9.53 -> 10.7 mm
Other:
- board size 63.2 x 45.7 mm -> 63.5 x 45.7 mm
